Commit message: fix: close phase 1 tf handoff and sensor output baseline

File: go2w_description/urdf/go2w_placeholder.urdf (robot description, URDF)
Before this commit: robot go2w_placeholder, 7 links, 6 joints
Links:
- added link imu_link, mass 0.05; collision box size=0.03 0.03 0.02; visual box size=0.03 0.03 0.02
- added link lidar_link, mass 0.2; collision cylinder length=0.05 radius=0.035; visual cylinder length=0.05 radius=0.035
Joints:
- added joint imu_joint: type fixed, parent sensor_mount_link, child imu_link, origin xyz=-0.02 0 0.0 rpy=0 0 0
- added joint lidar_joint: type fixed, parent sensor_mount_link, child lidar_link, origin xyz=0.02 0 0.055 rpy=0 0 0
